File: Hardware/PPG-Module/Gamma-PPG-Module.brd (EAGLE design)
At the start: 0 parts

Commit message: Updated PPG module BOM and board/schematic.  Note:  the board and schematic were taken directly from the Kick Jr repository without modification
Parts:
- added C1: 2.2u, CalvEngIO-Passives:C0603
- added J1: (no value), LinnesLab-Connectors:PPG.MODULE.2
- added LED1: (no value), LinnesLab-LED:LED-0805
- added PD: (no value), CalvEngIO-Sensors:2-SMD.GULLWING
- added U$3: LINNES.LAB.LOGO, CalvEngIO-Logos:LINNES.LAB.LOGO
Connections:
- new net GND: C1.2, J1.GND, PD.+
- new net LED.C: J1.LD1, LED1.C
- new net PD.C: J1.PD, PD.-
- new net V+: C1.1, J1.V+, LED1.A
Routing:
- net LED.C: track 0.00 -> 7.32 mm
- net PD.C: track 0.00 -> 4.92 mm
- net V+: track 0.00 -> 3.47 mm
- added copper zone on layer 1, net GND
- added copper zone on layer 16, net GND
Other:
- board outline added: 12.4 x 12.4 mm
