File: Hardware/PPG-Module/Gamma-PPG-Module.sch (EAGLE design)
At the start: 0 parts

Commit message: Updated PPG module BOM and board/schematic.  Note:  the board and schematic were taken directly from the Kick Jr repository without modification
Parts:
- added C1: 2.2u, CalvEngIO-Passives:CAPACITOR0603
- added J1: (no value), LinnesLab-Connectors:PPG.MODULE.2
- added LED1: (no value), LinnesLab-LED:LED0805
- added PD: (no value), CalvEngIO-Sensors:PHOTODIODE.-SMD.GULLWING
- added U$3: LINNES.LAB.LOGO, CalvEngIO-Logos:LINNES.LAB.LOGO
Connections:
- new net GND: C1.2, J1.GND, PD.A
- new net LED.C: J1.LD1.C, LED1.C
- new net PD.C: J1.PD.C, PD.C
- new net V+: C1.1, J1.V+, LED1.A
Other:
- note added: "(C) Linnes Lab, 2018 Purdue University Adapted for Purdue Milestones"
- note added: "Kick LL Jr: PPG Module"
