File: Hardware/Top/Gamma-TOP-OLD.sch (EAGLE design)
At the start: 63 parts, among them SW1 SWITCH.MOM, SW2 SWITCH.MOM, U1 FT231XS, U3 NRF52832_MODULE_MDBT42, U5 FT24C64A, Y1 32.768kHz

Commit message: Updated file names and completed preliminary BOM for each board
Parts:
- removed C18, C21: 120p, LinnesLab-Passives:CAPACITOR0603
- removed C19: 100n, LinnesLab-Passives:CAPACITOR0603
- removed NFCANTENNA: 2.1 uH, NFC-Antenna:MOLEX-1462360151-ANTENNA
- removed U5: FT24C64A, LinnesLab-DigitalIC:FT24C64A
Connections:
- removed net WP: U3.P0.02/AIN0, U5.WP
- net 3.3V: no longer C19.1, U5.VCC
- net GND: no longer C18.2, C19.2, C21.2, U5.GND
- net P0.09/NFC1: no longer C18.1, NFCANTENNA.NFC1
- net P0.10/NFC2: no longer C21.1, NFCANTENNA.NFC2
- net SCL: no longer U5.SCL
- net SDA: no longer U5.SDA
Other:
- note added: "Gamma Top Version A"
- note removed: "EEPROM Storage"
- note removed: "Gamma Top Version B (Full Version)"
- note removed: "NFC Tuning Circuit with Antenna"
Changed lines of the file:
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@@
 <part name="SUPPLY8" library="LinnesLab-Symbols" deviceset="3.3V" device=""/>
 <part name="GND6" library="LinnesLab-Symbols" deviceset="GND" device=""/>
-<part name="U5" library="LinnesLab-DigitalIC" deviceset="FT24C64A" device="" package3d_urn="urn:adsk.eagle:package:18172171/2"/>
-<part name="SUPPLY10" library="LinnesLab-Symbols" deviceset="3.3V" device=""/>
-<part name="GND5" library="LinnesLab-Symbols" deviceset="GND" device=""/>
-<part name="C19" library="LinnesLab-Passives" deviceset="CAPACITOR" device="0603" package3d_urn="urn:adsk.eagle:package:15661989/2" value="100n"/>
-<part name="SUPPLY11" library="LinnesLab-Symbols" deviceset="3.3V" device=""/>
-<part name="GND13" library="LinnesLab-Symbols" deviceset="GND" device=""/>
-<part name="NFCANTENNA" library="NFC-Antenna" deviceset="MOLEX-1462360151-ANTENNA" device="" value="2.1 uH"/>
-<part name="GND2" library="LinnesLab-Symbols" deviceset="GND" device=""/>
-<part name="GND4" library="LinnesLab-Symbols" deviceset="GND" device=""/>
-<part name="C18" library="LinnesLab-Passives" deviceset="CAPACITOR" device="0603" package3d_urn="urn:adsk.eagle:package:15661989/2" value="120p"/>
-<part name="C21" library="LinnesLab-Passives" deviceset="CAPACITOR" device="0603" package3d_urn="urn:adsk.eagle:package:15661989/2" value="120p"/>
 </parts>
 <sheets>
@@
 <wire x1="360.68" y1="68.58" x2="261.62" y2="68.58" width="0.1524" layer="97" style="dashdot"/>
 <wire x1="261.62" y1="142.24" x2="360.68" y2="142.24" width="0.1524" layer="97" style="dashdot"/>
-<text x="35.56" y="205.74" size="10.16" layer="90">Gamma Top Version B (Full Version)</text>
-<text x="-30.48" y="-43.18" size="5.08" layer="90">EEPROM Storage</text>
-<text x="269.24" y="-50.8" size="4.572" layer="90">NFC Tuning Circuit with Antenna</text>
+<text x="35.56" y="205.74" size="10.16" layer="90">Gamma Top Version A</text>
 </plain>
 <instances>
@@
 <instance part="GND6" gate="G$1" x="-195.58" y="58.42" smashed="yes">
 <attribute name="VALUE" x="-195.58" y="58.166" size="1.778" layer="96" align="top-center"/>
-</instance>
-<instance part="U5" gate="G$1" x="-10.16" y="-78.74" smashed="yes">
-<attribute name="NAME" x="-17.78" y="-72.39" size="1.778" layer="95"/>
-<attribute name="VALUE" x="-17.78" y="-86.36" size="1.778" layer="96"/>
-</instance>
-<instance part="SUPPLY10" gate="G$1" x="2.54" y="-73.66" smashed="yes">
-<attribute name="VALUE" x="2.54" y="-70.866" size="1.778" layer="96" align="bottom-center"/>
-</instance>
-<instance part="GND5" gate="G$1" x="2.54" y="-86.36" smashed="yes">
-<attribute name="VALUE" x="2.54" y="-86.614" size="1.778" layer="96" align="top-center"/>
-</instance>
-<instance part="C19" gate="G$1" x="10.16" y="-78.74" smashed="yes">
-<attribute name="NAME" x="11.684" y="-75.819" size="1.778" layer="95"/>
-<attribute name="VALUE" x="11.684" y="-80.899" size="1.778" layer="96"/>
-</instance>
-<instance part="SUPPLY11" gate="G$1" x="10.16" y="-71.12" smashed="yes">
-<attribute name="VALUE" x="10.16" y="-68.326" size="1.778" layer="96" align="bottom-center"/>
-</instance>
-<instance part="GND13" gate="G$1" x="10.16" y="-86.36" smashed="yes">
-<attribute name="VALUE" x="10.16" y="-86.614" size="1.778" layer="96" align="top-center"/>
-</instance>
-<instance part="NFCANTENNA" gate="G$1" x="304.8" y="-101.6" smashed="yes" rot="R90">
-<attribute name="NAME" x="294.64" y="-111.76" size="1.778" layer="95" rot="R90"/>
-<attribute name="VALUE" x="317.5" y="-111.76" size="1.778" layer="96" rot="R90"/>
-</instance>
-<instance part="GND2" gate="G$1" x="340.36" y="-86.36" smashed="yes">
-<attribute name="VALUE" x="340.36" y="-86.614" size="1.778" layer="96" align="top-center"/>
-</instance>
-<instance part="GND4" gate="G$1" x="299.72" y="-83.82" smashed="yes">
-<attribute name="VALUE" x="299.72" y="-84.074" size="1.778" layer="96" align="top-center"/>
-</instance>
-<instance part="C18" gate="G$1" x="294.64" y="-78.74" smashed="yes" rot="R90">
-<attribute name="NAME" x="291.719" y="-77.216" size="1.778" layer="95" rot="R90"/>
-<attribute name="VALUE" x="296.799" y="-77.216" size="1.778" layer="96" rot="R90"/>
-</instance>
-<instance part="C21" gate="G$1" x="337.82" y="-78.74" smashed="yes" rot="R90">
-<attribute name="NAME" x="334.899" y="-77.216" size="1.778" layer="95" rot="R90"/>
-<attribute name="VALUE" x="339.979" y="-77.216" size="1.778" layer="96" rot="R90"/>
 </instance>
 </instances>
@@
 <pinref part="GND6" gate="G$1" pin="GND"/>
 </segment>
-<segment>
-<pinref part="U5" gate="G$1" pin="GND"/>
-<wire x1="0" y1="-81.28" x2="2.54" y2="-81.28" width="0.1524" layer="91"/>
-<wire x1="2.54" y1="-81.28" x2="2.54" y2="-83.82" width="0.1524" layer="91"/>
-<pinref part="GND5" gate="G$1" pin="GND"/>
-</segment>
-<segment>
-<pinref part="C19" gate="G$1" pin="2"/>
-<pinref part="GND13" gate="G$1" pin="GND"/>
-<wire x1="10.16" y1="-83.82" x2="10.16" y2="-81.28" width="0.1524" layer="91"/>
-</segment>
-<segment>
-<pinref part="C18" gate="G$1" pin="2"/>
-<pinref part="GND4" gate="G$1" pin="GND"/>
-<wire x1="297.18" y1="-78.74" x2="299.72" y2="-78.74" width="0.1524" layer="91"/>
-<wire x1="299.72" y1="-78.74" x2="299.72" y2="-81.28" width="0.1524" layer="91"/>
-</segment>
-<segment>
-<pinref part="C21" gate="G$1" pin="2"/>
-<pinref part="GND2" gate="G$1" pin="GND"/>
-<wire x1="340.36" y1="-78.74" x2="340.36" y2="-83.82" width="0.1524" layer="91"/>
-</segment>
 </net>
 <net name="SWDIO" class="0">
@@
 <pinref part="SUPPLY8" gate="G$1" pin="3.3V"/>
 </segment>
-<segment>
-<pinref part="U5" gate="G$1" pin="VCC"/>
-<wire x1="0" y1="-76.2" x2="2.54" y2="-76.2" width="0.1524" layer="91"/>
-<wire x1="2.54" y1="-76.2" x2="2.54" y2="-73.66" width="0.1524" layer="91"/>
-<pinref part="SUPPLY10" gate="G$1" pin="3.3V"/>
-</segment>
-<segment>
-<pinref part="C19" gate="G$1" pin="1"/>
-<pinref part="SUPPLY11" gate="G$1" pin="3.3V"/>
-<wire x1="10.16" y1="-73.66" x2="10.16" y2="-71.12" width="0.1524" layer="91"/>
-</segment>
 </net>
 <net name="SDA" class="0">
@@
 <label x="-190.5" y="66.04" size="1.27" layer="95" xref="yes"/>
 </segment>
-<segment>
-<pinref part="U5" gate="G$1" pin="SDA"/>
-<wire x1="-22.86" y1="-76.2" x2="-20.32" y2="-76.2" width="0.1524" layer="91"/>
-<label x="-22.86" y="-76.2" size="1.27" layer="95" rot="R180" xref="yes"/>
-</segment>
 </net>
 <net name="SCL" class="0">
@@
 <wire x1="-198.12" y1="68.58" x2="-190.5" y2="68.58" width="0.1524" layer="91"/>
 <label x="-190.5" y="68.58" size="1.27" layer="95" xref="yes"/>
-</segment>
-<segment>
-<pinref part="U5" gate="G$1" pin="SCL"/>
-<wire x1="-22.86" y1="-78.74" x2="-20.32" y2="-78.74" width="0.1524" layer="91"/>
-<label x="-22.86" y="-78.74" size="1.27" layer="95" rot="R180" xref="yes"/>
 </segment>
 </net>
@@
 <label x="101.6" y="48.26" size="1.27" layer="95" rot="R180" xref="yes"/>
 </segment>
-<segment>
-<wire x1="287.02" y1="-60.96" x2="287.02" y2="-78.74" width="0.1524" layer="91"/>
-<label x="287.02" y="-60.96" size="4.572" layer="95" rot="R180" xref="yes"/>
-<pinref part="C18" gate="G$1" pin="1"/>
-<wire x1="287.02" y1="-78.74" x2="289.56" y2="-78.74" width="0.1524" layer="91"/>
-<wire x1="289.56" y1="-78.74" x2="289.56" y2="-91.44" width="0.1524" layer="91"/>
-<wire x1="289.56" y1="-91.44" x2="302.26" y2="-91.44" width="0.1524" layer="91"/>
-<pinref part="NFCANTENNA" gate="G$1" pin="NFC1"/>
-<wire x1="302.26" y1="-91.44" x2="302.26" y2="-96.52" width="0.1524" layer="91"/>
-</segment>
 </net>
 <net name="SCK" class="0">
@@
 <pinref part="U3" gate="G$1" pin="P0.10"/>
 <label x="104.14" y="48.26" size="1.27" layer="95" xref="yes"/>
-</segment>
-<segment>
-<wire x1="332.74" y1="-60.96" x2="332.74" y2="-78.74" width="0.1524" layer="91"/>
-<label x="332.74" y="-60.96" size="4.572" layer="95" rot="R180" xref="yes"/>
-<pinref part="NFCANTENNA" gate="G$1" pin="NFC2"/>
-<pinref part="C21" gate="G$1" pin="1"/>
-<wire x1="307.34" y1="-96.52" x2="332.74" y2="-96.52" width="0.1524" layer="91"/>
-<wire x1="332.74" y1="-96.52" x2="332.74" y2="-78.74" width="0.1524" layer="91"/>
 </segment>
 </net>
@@
 </segment>
 </net>
-<net name="WP" class="0">
-<segment>
-<pinref part="U5" gate="G$1" pin="WP"/>
-<wire x1="-22.86" y1="-81.28" x2="-20.32" y2="-81.28" width="0.1524" layer="91"/>
-<label x="-22.86" y="-81.28" size="1.27" layer="95" rot="R180" xref="yes"/>
-</segment>
-<segment>
-<pinref part="U3" gate="G$1" pin="P0.02/AIN0"/>
-<wire x1="83.82" y1="66.04" x2="83.82" y2="63.5" width="0.1524" layer="91"/>
-<label x="83.82" y="63.5" size="1.27" layer="95" rot="R270" xref="yes"/>
-</segment>
-</net>
