File: Hardware/Top/Basic/Gamma-TOP.brd (EAGLE design)
At the start: 38 x 38 mm, 58 parts, among them SW1 SWITCH.MOM, SW2 SWITCH.MOM, U1 FT231XS, U3 NRF52832_MODULE_MDBT42, Y1 32.768kHz

Commit message: small fixes
Connections:
- net GND: no longer SW1.B2, SW2.B2
Changed lines of the file:
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@@
 <?xml version="1.0" encoding="utf-8"?>
 <!DOCTYPE eagle SYSTEM "eagle.dtd">
-<eagle version="9.5.2">
+<eagle version="9.6.2">
 <drawing>
 <settings>
@@
 <layer number="25" name="tNames" color="7" fill="1" visible="yes" active="yes"/>
 <layer number="26" name="bNames" color="7" fill="1" visible="yes" active="yes"/>
-<layer number="27" name="tValues" color="7" fill="1" visible="yes" active="yes"/>
-<layer number="28" name="bValues" color="7" fill="1" visible="yes" active="yes"/>
+<layer number="27" name="tValues" color="7" fill="1" visible="no" active="yes"/>
+<layer number="28" name="bValues" color="7" fill="1" visible="no" active="yes"/>
 <layer number="29" name="tStop" color="7" fill="3" visible="no" active="yes"/>
 <layer number="30" name="bStop" color="7" fill="6" visible="no" active="yes"/>
@@
 <contactref element="R11" pad="1"/>
 <contactref element="CHRG1" pad="2"/>
-<contactref element="SW1" pad="B2"/>
 <contactref element="SW1" pad="B1"/>
 <contactref element="SW2" pad="B1"/>
-<contactref element="SW2" pad="B2"/>
 <contactref element="JP1" pad="1"/>
 <contactref element="C3" pad="1"/>
@@
 <wire x1="22.8954" y1="33.518" x2="23.6728" y2="32.7406" width="0.4572" layer="1"/>
 <via x="23.6728" y="32.7406" extent="1-16" drill="0.35"/>
-<wire x1="25.9714" y1="1.6616" x2="28.1814" y2="1.7124" width="0" layer="19" extent="1-1"/>
-<wire x1="18.0214" y1="1.6616" x2="16.3576" y2="4.572" width="0" layer="19" extent="1-1"/>
 </signal>
 <signal name="SWDIO">
