File: Hardware/Top/Plus/Gamma-TOP.sch (EAGLE design)
At the start: 63 parts, among them SW1 SWITCH.MOM, SW2 SWITCH.MOM, U1 FT231XS, U3 NRF52832_MODULE_MDBT42, U5 FT24C64A, Y1 32.768kHz

Commit message: small fixes
Connections:
- net GND: no longer SW1.4, SW2.4
Changed lines of the file:
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@@
 <?xml version="1.0" encoding="utf-8"?>
 <!DOCTYPE eagle SYSTEM "eagle.dtd">
-<eagle version="9.5.2">
+<eagle version="9.6.2">
 <drawing>
 <settings>
@@
 <segment>
 <pinref part="GND1" gate="G$1" pin="GND"/>
-<pinref part="SW1" gate="G$1" pin="4"/>
-<wire x1="307.34" y1="165.1" x2="304.8" y2="165.1" width="0.1524" layer="91"/>
 <pinref part="SW1" gate="G$1" pin="3"/>
 <wire x1="304.8" y1="167.64" x2="307.34" y2="167.64" width="0.1524" layer="91"/>
@@
 <pinref part="GND3" gate="G$1" pin="GND"/>
 <wire x1="347.98" y1="167.64" x2="347.98" y2="165.1" width="0.1524" layer="91"/>
-<pinref part="SW2" gate="G$1" pin="4"/>
-<wire x1="347.98" y1="165.1" x2="345.44" y2="165.1" width="0.1524" layer="91"/>
-</segment>
-<segment>
+</segment>
+<segment>
